File: projects/2CQ/hardware/2CQ/2CQ.kicad_pcb (KiCad board)
At the start: 2 copper layers, 17 parts, among them SW1 TOGGLE_ON-ON, U1 ES_DAISY_PATCH_SM_REV1

Commit message: Restart PCB
Parts:
- removed DS1: ~, 128x64_0.96_Disp_Module:128x64_0.96_Disp_Module
- removed EP1: EURORACK_POWERHEADER, ES_Daisy_Patch_SM_FB_Rev1:EURORACK_POWER_SHROUD_LOCK
- removed J_CV1, J_CV2, J_CV3, J_CV4, J_CV5, J_CV6, J_CV7, J_CV8: EURO_JACK, ES_Daisy_Patch_SM_FB_Rev1:S_JACK
- removed S1: TAC_SWITCH_PTH, ES_Daisy_Patch_SM_FB_Rev1:TL1105SPF250Q_SILK
- removed SW1: TOGGLE_ON-ON, ES_Daisy_Patch_SM_FB_Rev1:TOGGLE_ON-ON
- removed U1: ES_DAISY_PATCH_SM_REV1, ES_Daisy_Patch_SM_FB_Rev1:ES_DAISY_PATCH_SM_REV1
- removed VR1, VR2, VR3, VR4: M-10K-B-D, ES_Daisy_Patch_SM_FB_Rev1:9MM_SNAP-IN_POT_SILK
