File: projects/2CQ/hardware/2CQ/2CQ.kicad_pcb (KiCad board)
At the start: 2 copper layers, 0 parts

Commit message: Imported PCB settings from https://github.com/sethhillbrand/kicad_templates/tree/master/JLCPCB_1-2Layer
Other:
- copper layers 2 -> 4
Changed lines of the file:
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@@
 	(generator_version "8.0")
 	(general
-		(thickness 1.6)
+		(thickness 1.600198)
 		(legacy_teardrops no)
 	)
@@
 	)
 	(layers
-		(0 "F.Cu" signal)
-		(31 "B.Cu" signal)
-		(32 "B.Adhes" user "B.Adhesive")
-		(33 "F.Adhes" user "F.Adhesive")
+		(0 "F.Cu" signal "Front")
+		(1 "In1.Cu" signal)
+		(2 "In2.Cu" signal)
+		(31 "B.Cu" signal "Back")
 		(34 "B.Paste" user)
 		(35 "F.Paste" user)
@@
 		(38 "B.Mask" user)
 		(39 "F.Mask" user)
-		(40 "Dwgs.User" user "User.Drawings")
-		(41 "Cmts.User" user "User.Comments")
-		(42 "Eco1.User" user "User.Eco1")
-		(43 "Eco2.User" user "User.Eco2")
 		(44 "Edge.Cuts" user)
 		(45 "Margin" user)
 		(46 "B.CrtYd" user "B.Courtyard")
 		(47 "F.CrtYd" user "F.Courtyard")
-		(48 "B.Fab" user)
 		(49 "F.Fab" user)
-		(50 "User.1" user)
-		(51 "User.2" user)
-		(52 "User.3" user)
-		(53 "User.4" user)
-		(54 "User.5" user)
-		(55 "User.6" user)
-		(56 "User.7" user)
-		(57 "User.8" user)
-		(58 "User.9" user)
 	)
 	(setup
@@
 			(layer "dielectric 1"
 				(type "core")
-				(thickness 1.51)
+				(thickness 0.480066)
+				(material "FR4")
+				(epsilon_r 4.5)
+				(loss_tangent 0.02)
+			)
+			(layer "In1.Cu"
+				(type "copper")
+				(thickness 0.035)
+			)
+			(layer "dielectric 2"
+				(type "prepreg")
+				(thickness 0.480066)
+				(material "FR4")
+				(epsilon_r 4.5)
+				(loss_tangent 0.02)
+			)
+			(layer "In2.Cu"
+				(type "copper")
+				(thickness 0.035)
+			)
+			(layer "dielectric 3"
+				(type "core")
+				(thickness 0.480066)
 				(material "FR4")
 				(epsilon_r 4.5)
@@
 		)
 		(pad_to_mask_clearance 0)
+		(solder_mask_min_width 0.12)
 		(allow_soldermask_bridges_in_footprints no)
 		(pcbplotparams

Commit message: Added model to thonk jack
Parts:
- added DS1: SSD1306_96_128_64_7P, 2CQ:128x64_0.96_Disp_Module, F.Cu at (128.9, 124.9)
- added EP1: EURORACK_POWERHEADER, ES_Daisy_Patch_SM_FB_Rev1:EURORACK_POWER_SHROUD_LOCK, F.Cu at (78.4, 116.4)
- added J_CV1: EURO_JACK, ES_Daisy_Patch_SM_FB_Rev1:S_JACK, F.Cu at (74.3, 48.1)
- added J_CV2: EURO_JACK, ES_Daisy_Patch_SM_FB_Rev1:S_JACK, F.Cu at (84.4, 48.1)
- added J_CV3: EURO_JACK, ES_Daisy_Patch_SM_FB_Rev1:S_JACK, F.Cu at (94.5, 48.1)
- added J_CV4: EURO_JACK, ES_Daisy_Patch_SM_FB_Rev1:S_JACK, F.Cu at (104.7, 48.1)
- added J_CV5: EURO_JACK, ES_Daisy_Patch_SM_FB_Rev1:S_JACK, F.Cu at (114.8, 48.1)
- added J_CV6: EURO_JACK, ES_Daisy_Patch_SM_FB_Rev1:S_JACK, F.Cu at (124.9, 48.1)
- added J_CV7: EURO_JACK, ES_Daisy_Patch_SM_FB_Rev1:S_JACK, F.Cu at (135.1, 48.1)
- added J_CV8: EURO_JACK, ES_Daisy_Patch_SM_FB_Rev1:S_JACK, F.Cu at (145.2, 48.1)
- added S1: TAC_SWITCH_PTH, ES_Daisy_Patch_SM_FB_Rev1:TL1105SPF250Q_SILK, F.Cu at (104.5, 117.0)
- added SW1: TOGGLE_ON-ON, ES_Daisy_Patch_SM_FB_Rev1:TOGGLE_ON-ON, F.Cu at (93.3, 115.6)
- added U1: ES_DAISY_PATCH_SM_REV1, ES_Daisy_Patch_SM_FB_Rev1:ES_DAISY_PATCH_SM_REV1, F.Cu at (103.8, 76.5)
- added VR1: M-10K-B-D, ES_Daisy_Patch_SM_FB_Rev1:9MM_SNAP-IN_POT_SILK, F.Cu at (76.6, 103.1)
- added VR2: M-10K-B-D, ES_Daisy_Patch_SM_FB_Rev1:9MM_SNAP-IN_POT_SILK, F.Cu at (91.3, 103.1)
- added VR3: M-10K-B-D, ES_Daisy_Patch_SM_FB_Rev1:9MM_SNAP-IN_POT_SILK, F.Cu at (106.0, 103.1)
- added VR4: M-10K-B-D, ES_Daisy_Patch_SM_FB_Rev1:9MM_SNAP-IN_POT_SILK, F.Cu at (120.8, 103.1)

Commit message: Added 3d models and updated PCB
Parts:
- moved J_CV1 99.8 mm to (82.4, 147.6)
- moved J_CV2 99.8 mm to (92.5, 147.6)
- moved J_CV3 99.8 mm to (102.6, 147.6)
- moved J_CV4 99.8 mm to (112.8, 147.6)
- moved J_CV7 91.4 mm to (102.6, 133.6)
- moved J_CV5 91.4 mm to (82.4, 133.6)
- moved J_CV6 91.4 mm to (92.5, 133.6)
- moved J_CV8 91.4 mm to (112.8, 133.6)
- moved DS1 69.0 mm to (84.4, 72.2)
- moved SW1 33.7 mm to (96.8, 82.0), turned to 90 degrees
- moved VR2 28.4 mm to (108.9, 80.8)
- moved VR1 23.8 mm to (85.0, 80.8)
- moved VR3 21.7 mm to (85.3, 96.5)
- moved S1 21.6 mm to (97.6, 96.5)
- moved EP1 19.4 mm to (97.6, 113.3), turned to -90 degrees
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Other:
- board outline added: 48.5 x 111 mm

Commit message: moved power
Parts:
- moved EP1 9.02 mm to (97.3, 122.3), turned to 0 degrees
- moved DS1 0.25 mm to (84.4, 72.5)

Commit message: PCB Stuff
Parts:
- moved EP1 11.2 mm to (86.1, 122.3), turned to 180 degrees
- moved S1 10.1 mm to (98.0, 106.7)
- moved SW1 8.13 mm to (97.0, 90.2), turned to 180 degrees
Other:
- board text added: "-12V"

Commit message: Moving shit around
Parts:
- moved J_CV5 1.52 mm to (82.4, 132.1)
- moved J_CV6 1.52 mm to (92.5, 132.1)
- moved J_CV7 1.52 mm to (102.6, 132.1)
- moved J_CV8 1.52 mm to (112.8, 132.1)
- moved J_CV1 1.02 mm to (82.4, 146.6)
- moved J_CV2 1.02 mm to (92.5, 146.6)
- moved J_CV3 1.02 mm to (102.6, 146.6)
- moved J_CV4 1.02 mm to (112.8, 146.6)
- moved EP1 0.57 mm to (86.4, 121.8)
Routing:
- added copper zone on B.Cu, net GND
- added copper zone on F.Cu, net GND
Other:
- copper layers 4 -> 2
Changed lines of the file:
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@@
 	(layers
 		(0 "F.Cu" signal "Front")
-		(1 "In1.Cu" signal)
-		(2 "In2.Cu" signal)
 		(31 "B.Cu" signal "Back")
 		(34 "B.Paste" user)
@@
 			(layer "dielectric 1"
 				(type "core")
-				(thickness 0.480066)
-				(material "FR4")
-				(epsilon_r 4.5)
-				(loss_tangent 0.02)
-			)
-			(layer "In1.Cu"
-				(type "copper")
-				(thickness 0.035)
-			)
-			(layer "dielectric 2"
-				(type "prepreg")
-				(thickness 0.480066)
-				(material "FR4")
-				(epsilon_r 4.5)
-				(loss_tangent 0.02)
-			)
-			(layer "In2.Cu"
-				(type "copper")
-				(thickness 0.035)
-			)
-			(layer "dielectric 3"
-				(type "core")
-				(thickness 0.480066)
+				(thickness 1.510198)
 				(material "FR4")
 				(epsilon_r 4.5)
@@
 	(footprint "ES_Daisy_Patch_SM_FB_Rev1:S_JACK"
 		(layer "F.Cu")
-		(at 92.522 133.604)
+		(at 92.522 132.08)
 		(property "Reference" "J_CV6"
 			(at -4.7498 4.4704 90)
@@
 	(footprint "ES_Daisy_Patch_SM_FB_Rev1:S_JACK"
 		(layer "F.Cu")
-		(at 102.649 147.574)
+		(at 102.649 146.558)
 		(property "Reference" "J_CV3"
 			(at -4.7498 4.4704 90)
@@
 	(footprint "ES_Daisy_Patch_SM_FB_Rev1:S_JACK"
 		(layer "F.Cu")
-		(at 102.649 133.604)
+		(at 102.649 132.08)
 		(property "Reference" "J_CV7"
 			(at -4.7498 4.4704 90)
@@
 	(footprint "ES_Daisy_Patch_SM_FB_Rev1:S_JACK"
 		(layer "F.Cu")
-		(at 82.395 133.604)
+		(at 82.395 132.08)
 		(property "Reference" "J_CV5"
 			(at -4.7498 4.4704 90)
@@
 	(footprint "ES_Daisy_Patch_SM_FB_Rev1:S_JACK"
 		(layer "F.Cu")
-		(at 82.395 147.574)
+		(at 82.395 146.558)
 		(property "Reference" "J_CV1"
 			(at -4.7498 4.4704 90)
@@
 	(footprint "ES_Daisy_Patch_SM_FB_Rev1:S_JACK"
 		(layer "F.Cu")
-		(at 112.776 147.574)
+		(at 112.776 146.558)
 		(property "Reference" "J_CV4"
 			(at -4.7498 4.4704 90)
@@
 	(footprint "ES_Daisy_Patch_SM_FB_Rev1:EURORACK_POWER_SHROUD_LOCK"
 		(layer "F.Cu")
-		(at 86.106 122.301 180)
+		(at 86.36 121.793 180)
 		(property "Reference" "EP1"
 			(at 0 0 360)
@@
 			(size 2.5 2.5)
 			(drill 2)
-			(layers "F&B.Cu" "*.Mask")
+			(layers "*.Cu" "*.Mask")
 		)
 		(pad "" np_thru_hole circle
@@
 			(size 2.5 2.5)
 			(drill 2)
-			(layers "F&B.Cu" "*.Mask")
+			(layers "*.Cu" "*.Mask")
 		)
 		(pad "" np_thru_hole circle
@@
 			(size 2.5 2.5)
 			(drill 2)
-			(layers "F&B.Cu" "*.Mask")
+			(layers "*.Cu" "*.Mask")
 		)
 		(pad "" np_thru_hole circle
@@
 			(size 2.5 2.5)
 			(drill 2)
-			(layers "F&B.Cu" "*.Mask")
+			(layers "*.Cu" "*.Mask")
 		)
 		(pad "1" thru_hole rect
@@
 	(footprint "ES_Daisy_Patch_SM_FB_Rev1:S_JACK"
 		(layer "F.Cu")
-		(at 92.522 147.574)
+		(at 92.522 146.558)
 		(property "Reference" "J_CV2"
 			(at -4.7498 4.4704 90)
@@
 	(footprint "ES_Daisy_Patch_SM_FB_Rev1:S_JACK"
 		(layer "F.Cu")
-		(at 112.776 133.604)
+		(at 112.776 132.08)
 		(property "Reference" "J_CV8"
 			(at -4.7498 4.4704 90)
@@
 		)
 	)
+	(zone
+		(net 2)
+		(net_name "GND")
+		(layers "F&B.Cu")
+		(hatch edge 0.5)
+		(connect_pads
+			(clearance 0.5)
+		)
+		(min_thickness 0.25)
+		(filled_areas_thickness no)
+		(fill yes
+			(thermal_gap 0.5)
+			(thermal_bridge_width 0.5)
+		)
+		(polygon
+			(pts
+				(xy 66.802 40.894) (xy 128.524 41.148) (xy 129.794 159.258) (xy 67.818 160.02)
+			)
+		)
+	)
